File: clip.kicad_pcb (KiCad board)
At the start: 2 copper layers, 47 parts, among them J1 LiPo, J2 USB_B_Micro, J3 BME680, J4 LIS3DH, J5 Conn_01x07, J6 Conn_01x18, J7 Conn_01x18, Q1 2.5A/30V, Q2 S8050, Q3 S8050, SW1 Switch, SW2 Switch, U1 MCP73831, U2 AP2112K-3.3, U3 FT231XS, U4 ESP32-WROOM-32

Commit message: Update design
Parts:
- removed D4: Green, LED_SMD:LED_0805_2012Metric_Pad1.15x1.40mm_HandSolder
- removed J5: Conn_01x07, Connector_PinHeader_2.54mm:PinHeader_1x07_P2.54mm_Vertical
- removed J6, J7: Conn_01x18, Connector_PinHeader_2.54mm:PinHeader_1x18_P2.54mm_Vertical
- removed R3: 1K, Resistor_SMD:R_0805_2012Metric_Pad1.15x1.40mm_HandSolder
- D1: value Red -> Green
- J2: footprint Connector_USB:USB_Micro-B_Amphenol_10103594-0001LF_Horizontal -> Connector_USB:USB_Micro-B_Wuerth_614105150721_Vertical
- moved SW1 78.4 mm to (131.3, 108.9), turned to 90 degrees
- moved C11 74.9 mm to (160.2, 122.8), turned to 270 degrees
- moved R11 71.7 mm to (135.3, 108.4), turned to 270 degrees
- moved J3 70.4 mm to (129.0, 98.1), turned to 90 degrees
- moved R8 69.5 mm to (144.7, 54.6), turned to 180 degrees
- moved C6 68.3 mm to (134.0, 77.5)
- moved R1 62.8 mm to (150.1, 63.1)
- moved C12 60.9 mm to (162.4, 108.4), turned to 90 degrees
- moved Q3 59.3 mm to (160.8, 83.7), turned to 270 degrees
- moved R6 58.7 mm to (145.6, 58.1)
- moved U1 58.6 mm to (139.4, 59.1)
- moved J2 58.4 mm to (127.8, 77.7), turned to 270 degrees
- moved C9 55.2 mm to (141.2, 79.8), turned to 270 degrees
- moved C2 54.9 mm to (145.6, 60.2)
- moved C10 54.6 mm to (162.4, 122.8), turned to 270 degrees
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Routing:
- net +3V3: track 0.00 -> 194.3 mm, vias 0 -> 4
- net GND: track 0.00 -> 110.2 mm, vias 0 -> 1
- net EN: track 0.00 -> 63.5 mm
- net SDA: track 0.00 -> 56.8 mm, vias 0 -> 1
- net SCL: track 0.00 -> 56.6 mm, vias 0 -> 2
- net VBUS: track 0.00 -> 54.8 mm, vias 0 -> 2
- net IO0: track 0.00 -> 48.5 mm
- net TX0: track 0.00 -> 46.1 mm, vias 0 -> 2
- net RX0: track 0.00 -> 39.8 mm, vias 0 -> 2
- net VIN: track 0.00 -> 28.5 mm, vias 0 -> 2
- net +BATT: track 0.00 -> 22.5 mm
- net Net-(C7-Pad1): track 0.00 -> 19.2 mm
- net Net-(R7-Pad2): track 0.00 -> 15.4 mm
- net Net-(R4-Pad2): track 0.00 -> 15.1 mm
- net Net-(R1-Pad1): track 0.00 -> 14.8 mm, vias 0 -> 2
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- added copper zone on B.Cu, net GND
- added copper zone on F.Cu, net GND
Other:
- board outline added: 50.5 x 80.7 mm
- net class +3V3 added: clearance 0.2, trace_width 0.5, via_dia 1.1, via_drill 0.7
- net class +BATT added: clearance 0.2, trace_width 0.5, via_dia 1.1, via_drill 0.7
- net class VBUS added: clearance 0.2, trace_width 0.5, via_dia 1.1, via_drill 0.7
- net class VIN added: clearance 0.2, trace_width 0.5, via_dia 1.1, via_drill 0.7

Commit message: Update design
Parts:
- moved C5 21.0 mm to (154.4, 76.8), turned to 270 degrees
- moved J2 20.4 mm to (147.5, 72.6), turned to 0 degrees
- moved R4 19.4 mm to (151.9, 76.9), turned to 270 degrees
- moved R7 11.7 mm to (145.6, 76.8), turned to 270 degrees
- moved C6 9.29 mm to (143.3, 76.8), turned to 270 degrees
- moved C8 3.78 mm to (143.3, 83.6)
- moved C9 3.78 mm to (141.1, 83.5)
- moved C7 3.75 mm to (153.4, 83.8)
- moved Q2 3.75 mm to (160.9, 79.6)
- moved Q3 3.75 mm to (160.8, 87.5)
- moved R12 3.75 mm to (162.6, 83.6)
- moved R13 3.75 mm to (159.1, 83.6)
- moved U3 3.75 mm to (148.4, 83.6)
- moved C4 3.66 mm to (159.3, 70.0)
- moved C3 2.73 mm to (150.4, 66.5)
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- renumbered SW1 to BOOT, SW2 to EN
Routing:
- net Net-(R7-Pad2): track 15.4 -> 3.04 mm
- net Net-(R4-Pad2): track 15.1 -> 7.53 mm
- net +3V3: track 194.3 -> 187.8 mm
- net VBUS: track 54.8 -> 49.8 mm, vias 2 -> 1
- net TX0: track 46.1 -> 42.0 mm
- net /D-: track 13.0 -> 9.35 mm
- net EN: track 63.5 -> 60.0 mm
- net IO0: track 48.5 -> 45.8 mm
- net GND: track 110.2 -> 107.9 mm
- net RX0: track 39.8 -> 42.0 mm
- net Net-(R5-Pad1): track 2.60 -> 3.69 mm
- net +BATT: track 22.5 -> 23.6 mm
- net VIN: track 28.5 -> 27.6 mm
- net Net-(R6-Pad1): track 3.20 -> 4.00 mm
- net /D+: track 13.1 -> 12.5 mm
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
Commit message: Refactor design
Parts:
- added J5: Moisture, Connector_PinHeader_2.54mm:PinHeader_1x03_P2.54mm_Horizontal, F.Cu at (146.2, 61.5)
- J2: footprint Connector_USB:USB_Micro-B_Wuerth_614105150721_Vertical -> Connector_USB:USB_Micro-B_Wuerth_629105150521
- JP1: footprint Connector_PinHeader_2.54mm:PinHeader_1x02_P2.54mm_Vertical -> Jumper:SolderJumper-2_P1.3mm_Open_TrianglePad1.0x1.5mm
- moved J2 22.9 mm to (128.3, 85.0), turned to 270 degrees
- moved C5 20.7 mm to (134.7, 83.1), turned to 90 degrees
- moved R8 16.7 mm to (160.0, 61.5)
- moved R4 16.2 mm to (137.0, 83.1), turned to 90 degrees
- moved C6 13.6 mm to (134.6, 87.3)
- moved R7 13.6 mm to (136.9, 87.2)
- moved D3 7.50 mm to (157.9, 54.6), turned to 180 degrees
- moved JP1 6.96 mm to (155.8, 61.5), turned to 180 degrees
- moved C2 6.81 mm to (146.2, 67.0)
- moved D1 6.81 mm to (150.6, 65.1)
- moved R1 6.81 mm to (150.7, 70.0)
- moved R6 6.81 mm to (146.2, 64.9)
- moved U1 6.81 mm to (139.7, 65.9)
- moved C3 6.81 mm to (150.7, 73.3)
- moved C4 6.81 mm to (159.6, 76.8)
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- renumbered BOOT to SW1, EN to SW2
Routing:
- net IO34: track 0.00 -> 88.9 mm, vias 0 -> 1
- net VBUS: track 49.8 -> 73.1 mm, vias 1 -> 0
- net GND: track 107.9 -> 118.5 mm, vias 1 -> 2
- net Net-(R7-Pad2): track 3.04 -> 12.8 mm
- net Net-(R4-Pad2): track 7.53 -> 12.7 mm
- net /D+: track 12.5 -> 7.78 mm
- net +3V3: track 187.8 -> 192.5 mm
- net Net-(D3-Pad2): track 3.38 -> 7.61 mm
- net Net-(D3-Pad1): track 3.81 -> 7.71 mm
- net RX0: track 42.0 -> 39.9 mm
- net TX0: track 42.0 -> 39.8 mm
- net ~RTS: track 11.8 -> 13.7 mm
- net +BATT: track 23.6 -> 21.9 mm
- net /D-: track 9.35 -> 7.79 mm
- net IO0: track 45.8 -> 45.1 mm
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
Commit message: Update design
Parts:
- removed the C5 at (134.7, 83.1)
- removed the C6 at (134.6, 87.3)
- removed the C7 at (153.5, 86.0)
- removed C8: 0.1uF/50V, Capacitor_SMD:C_0805_2012Metric_Pad1.15x1.40mm_HandSolder
- removed C9: 4.7uF/6.3V, Capacitor_SMD:C_0805_2012Metric_Pad1.15x1.40mm_HandSolder
- removed Q2, Q3: S8050, Package_TO_SOT_SMD:SOT-23
- removed R12, R13: 10K, Resistor_SMD:R_0805_2012Metric_Pad1.15x1.40mm_HandSolder
- removed the R4 at (137.0, 83.1)
- removed the R6 at (146.2, 64.9)
- removed the R7 at (136.9, 87.2)
- removed the U3 at (148.5, 85.8)
- added D4: Green, LED_SMD:LED_0805_2012Metric_Pad1.15x1.40mm_HandSolder, F.Cu at (155.7, 74.9)
- added J6: Conn_01x07, Connector_PinHeader_2.54mm:PinHeader_1x06_P2.54mm_Vertical, F.Cu at (142.6, 97.7)
- added J7: Conn_01x07, Connector_PinHeader_2.54mm:PinHeader_1x02_P2.54mm_Vertical, F.Cu at (140.1, 60.6)
- added J8: Conn_01x07, Connector_PinHeader_2.54mm:PinHeader_1x02_P2.54mm_Vertical, F.Cu at (171.4, 120.2)
- added R3: 1K, Resistor_SMD:R_0805_2012Metric_Pad1.15x1.40mm_HandSolder, F.Cu at (155.7, 79.9)
- added R5: 2.0K, Resistor_SMD:R_0805_2012Metric_Pad1.15x1.40mm_HandSolder, F.Cu at (146.6, 74.8)
- D1: value Green -> Red
- J2: footprint Connector_USB:USB_Micro-B_Wuerth_629105150521 -> Connector_USB:USB_Micro-B_Wuerth_614105150721_Vertical
- moved J2 32.0 mm to (140.1, 55.3), turned to 180 degrees
- moved R2 13.7 mm to (146.2, 64.4), turned to 180 degrees
- moved C2 9.91 mm to (146.6, 76.9)
- moved D1 9.91 mm to (151.0, 75.0)
- moved R1 9.91 mm to (151.1, 79.9)
- moved U1 9.91 mm to (140.1, 75.8)
- moved J4 6.32 mm to (150.9, 91.9)
- moved J3 6.28 mm to (129.0, 91.8)
- moved C3 5.90 mm to (150.6, 67.4)
- moved C4 5.90 mm to (159.6, 70.9)
- moved R4 5.90 mm to (159.6, 67.2)
- moved U2 5.90 mm to (154.7, 67.4)
- moved D2 5.77 mm to (146.3, 68.6)
- moved Q1 5.52 mm to (140.1, 67.8)
- moved C1 4.62 mm to (134.0, 71.2), turned to 90 degrees
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- renumbered C10 to C5, C11 to C6, C12 to C7, R5 to R4, R8 to R6, R11 to R7, R9 to R8, R10 to R9, U4 to U3
Connections:
- C5 pad 1: +3V3 -> Net-(C5-Pad1)
- C6 pad 1: +3V3 -> Net-(C5-Pad1)
- J1 pad 1: GND -> +BATT
- J1 pad 2: +BATT -> GND
- J2 pad 2: /D- -> Net-(J2-Pad2)
- J2 pad 3: /D+ -> Net-(J2-Pad3)
- U3 pad 2: +3V3 -> Net-(C5-Pad1)
Routing:
- net VBUS: track 73.1 -> 42.6 mm
- net IO0: track 45.1 -> 20.8 mm
- net Net-(C7-Pad1): track 19.2 -> 0.00 mm
- net GND: track 118.5 -> 100.1 mm, vias 2 -> 4
- net Net-(C5-Pad1): track 0.00 -> 14.8 mm
- net RX0: track 39.9 -> 25.9 mm, vias 2 -> 1
- net ~RTS: track 13.7 -> 0.00 mm
- net ~DTR: track 13.3 -> 0.00 mm
- net Net-(R7-Pad2): track 12.8 -> 0.00 mm
- net Net-(R4-Pad2): track 12.7 -> 0.00 mm
- net TX0: track 39.8 -> 28.4 mm, vias 2 -> 1
- net /D-: track 7.79 -> 0.00 mm
- net /D+: track 7.78 -> 0.00 mm
- net Net-(R1-Pad1): track 14.8 -> 22.2 mm
- net SDA: track 56.8 -> 50.3 mm
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
Commit message: Refactor design
Parts:
- moved R3 1.83 mm to (156.7, 78.3), turned to 270 degrees
- moved R1 1.82 mm to (152.1, 78.4), turned to 90 degrees
Routing:
- net Net-(D1-Pad1): track 5.54 -> 2.56 mm
- net Net-(D4-Pad2): track 4.95 -> 2.24 mm
- net Net-(R1-Pad1): track 22.2 -> 21.4 mm, vias 2 -> 0

Commit message: Update design
Parts:
- removed D3: Yellow, LED_SMD:LED_0805_2012Metric_Pad1.15x1.40mm_HandSolder
- removed J6: Conn_01x07, Connector_PinHeader_2.54mm:PinHeader_1x06_P2.54mm_Vertical
- removed J7: Conn_01x07, Connector_PinHeader_2.54mm:PinHeader_1x02_P2.54mm_Vertical
- added DL: Conn_01x07, Connector_PinHeader_2.54mm:PinHeader_1x02_P2.54mm_Vertical, F.Cu at (126.5, 120.2)
- added FW: Conn_01x07, Connector_PinHeader_2.54mm:PinHeader_1x06_P2.54mm_Vertical, F.Cu at (142.6, 97.7)
- added POWER: Yellow, LED_SMD:LED_0805_2012Metric_Pad1.15x1.40mm_HandSolder, F.Cu at (158.1, 54.6)
- added VIN: Conn_01x07, Connector_PinHeader_2.54mm:PinHeader_1x02_P2.54mm_Vertical, F.Cu at (140.0, 61.1)
- moved C5 2.28 mm to (164.7, 122.8)
- moved C6 2.18 mm to (162.4, 122.8)
- moved D1 2.02 mm to (152.3, 76.5)
- moved U2 2.02 mm to (154.8, 69.4)
- moved C3 1.94 mm to (150.7, 69.4)
- moved C4 1.94 mm to (159.6, 72.9)
- moved R4 1.94 mm to (159.6, 69.2)
- moved D4 1.93 mm to (156.8, 76.5)
- moved D2 1.89 mm to (146.3, 70.5)
- moved Q1 1.68 mm to (140.1, 69.5)
- moved R2 1.68 mm to (146.2, 66.1)
- moved R5 1.68 mm to (146.6, 76.5)
- moved U1 1.68 mm to (140.1, 77.5)
- moved C2 1.68 mm to (146.6, 78.6)
- moved C1 1.60 mm to (134.0, 72.8)
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- renumbered J1 to BATTERY, J3 to BME680, SW1 to BOOT, SW2 to EN, J4 to LIS3DH, J5 to MOISTURE, J8 to PW, J2 to USB
Routing:
- net IO0: track 20.8 -> 39.5 mm
- net SDA: track 50.3 -> 59.6 mm
- net GND: track 100.1 -> 106.5 mm
- net Net-(R1-Pad1): track 21.4 -> 24.5 mm
- net VBUS: track 42.6 -> 45.7 mm
- net RX0: track 25.9 -> 28.5 mm
- net IO34: track 91.0 -> 93.2 mm
- net SCL: track 56.1 -> 57.9 mm
- net +BATT: track 23.2 -> 24.9 mm
- net Net-(D3-Pad1): track 7.71 -> 8.48 mm
- net Net-(C5-Pad1): track 14.8 -> 15.5 mm
- net Net-(D3-Pad2): track 7.61 -> 8.26 mm
Other:
- board text added: "+"
- board text added: "3V3"
- board text added: "3Vo"
- board text added: "ADC"
- board text added: "CS"
- board text added: "EN"
- board text added: "G0"
- board text added: "GND"
- board text added: "INT"
- board text added: "RXD"
- board text added: "SCK"
- board text added: "SCL"
- board text added: "SDA"
- board text added: "SDI"
- board text added: "SDO"
- board text added: "TXD"
- board text added: "Vin"

Commit message: Update design
Parts:
- removed BME680: BME680, Connector_PinHeader_2.54mm:PinHeader_1x07_P2.54mm_Vertical
- removed C7: 0.1uF/50V, Capacitor_SMD:C_0805_2012Metric_Pad1.15x1.40mm_HandSolder
- removed DL, PW: Conn_01x07, Connector_PinHeader_2.54mm:PinHeader_1x02_P2.54mm_Vertical
- removed MOISTURE: Moisture, Connector_PinHeader_2.54mm:PinHeader_1x03_P2.54mm_Horizontal
- added BME1: BME680, Connector_PinHeader_2.54mm:PinHeader_1x07_P2.54mm_Vertical, F.Cu at (129.0, 90.7)
- added JP2: SJ, Jumper:SolderJumper-2_P1.3mm_Open_TrianglePad1.0x1.5mm, F.Cu at (166.7, 74.8)
- added MOISTURE1: MOISTURE, Connector_PinHeader_2.54mm:PinHeader_1x03_P2.54mm_Horizontal, F.Cu at (146.3, 61.1)
- D2: value 1A/23V/620mV -> Red; footprint Diode_SMD:D_SOD-323_HandSoldering -> LED_SMD:LED_0805_2012Metric_Pad1.15x1.40mm_HandSolder
- D3: renamed from POWER; value Yellow -> 1A/23V/620mV; footprint LED_SMD:LED_0805_2012Metric_Pad1.15x1.40mm_HandSolder -> Diode_SMD:D_SOD-323_HandSoldering
- R1: value 1K -> 10K
- R2: value 10K -> 1K
- R4: value 100K -> 1K
- R5: value 2.0K -> 100K
- R6: value 1K -> 1.0K
- USB1: renamed from USB; footprint Connector_USB:USB_Micro-B_Wuerth_614105150721_Vertical -> Connector_USB:USB_Micro-B_Wuerth_629105150521
- moved USB1 29.1 mm to (126.8, 81.2), turned to 270 degrees
- moved R6 22.3 mm to (148.3, 80.1), turned to 0 degrees
- moved D3 22.1 mm to (146.0, 73.2)
- moved VIN1 19.7 mm to (133.9, 79.9), turned to 0 degrees
- moved R2 18.3 mm to (154.0, 82.6), turned to 0 degrees
- moved R3 16.6 mm to (144.7, 67.2)
- moved R4 13.5 mm to (158.4, 82.7), turned to 180 degrees
- moved R5 13.5 mm to (159.4, 72.1), turned to 270 degrees
- moved C3 10.9 mm to (159.4, 75.9), turned to 270 degrees
- moved R1 10.3 mm to (142.3, 76.1), turned to 180 degrees
- moved C1 10.1 mm to (139.8, 81.1)
- moved C4 9.14 mm to (150.5, 72.3), turned to 90 degrees
- moved JP1 6.63 mm to (153.0, 67.1)
- moved U1 4.98 mm to (143.5, 81.1)
- moved R9 4.76 mm to (163.1, 108.4), turned to 90 degrees
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- renumbered BATTERY to BATTERY1, BOOT to BOOT1, EN to EN1, FW to FLASH1, LIS3DH to LIS1, VIN to VIN1
Connections:
- net CLK renamed Net-(U3-Pad20)
- net CMD renamed Net-(U3-Pad19)
- net IO12 renamed Net-(U3-Pad14)
- net IO13 renamed Net-(U3-Pad16)
- net IO14 renamed Net-(U3-Pad13)
- net IO15 renamed Net-(U3-Pad23)
- net IO16 renamed Net-(U3-Pad27)
- net IO17 renamed Net-(U3-Pad28)
- net IO18 renamed Net-(U3-Pad30)
- net IO19 renamed Net-(U3-Pad31)
- net IO23 renamed Net-(U3-Pad37)
- net IO25 renamed Net-(U3-Pad10)
- net IO26 renamed Net-(U3-Pad11)
- net IO27 renamed Net-(U3-Pad12)
- net IO32 renamed Net-(U3-Pad8)
- net IO35 renamed Net-(U3-Pad7)
- net IO4 renamed Net-(U3-Pad26)
- net IO5 renamed Net-(U3-Pad29)
- net SD0 renamed Net-(U3-Pad21)
- net SD1 renamed Net-(U3-Pad22)
- net SD2 renamed Net-(U3-Pad17)
- net SD3 renamed Net-(U3-Pad18)
- net VN renamed Net-(U3-Pad5)
- net VP renamed Net-(U3-Pad4)
- C3 pad 1: VIN -> Net-(C3-Pad1)
- C4 pad 1: +3V3 -> Net-(C4-Pad1)
- C5 pad 1: Net-(C5-Pad1) -> +3V3
- C6 pad 1: Net-(C5-Pad1) -> +3V3
- D2 pad 1: VIN -> Net-(D2-Pad1)
- D2 pad 2: VBUS -> Net-(D2-Pad2)
- D3 pad 1: Net-(D3-Pad1) -> Net-(C4-Pad1)
- D3 pad 2: Net-(D3-Pad2) -> VBUS
- JP1 pad 2: Net-(D3-Pad2) -> Net-(D2-Pad2)
- LIS1 pad 8: Net-(J4-Pad8) -> INT
- Q1 pad 2: VIN -> Net-(C4-Pad1)
- R1 pad 1: Net-(R1-Pad1) -> GND
- R1 pad 2: Net-(D1-Pad1) -> VBUS
- R2 pad 1: GND -> Net-(R2-Pad1)
- R2 pad 2: VBUS -> Net-(D1-Pad1)
- R3 pad 1: Net-(D4-Pad2) -> Net-(D2-Pad1)
- R3 pad 2: Net-(R1-Pad1) -> GND
- R4 pad 1: Net-(R4-Pad1) -> Net-(D4-Pad2)
- R4 pad 2: VIN -> Net-(R2-Pad1)
- R5 pad 2: GND -> Net-(C4-Pad1)
- R6 pad 1: Net-(D3-Pad1) -> Net-(R6-Pad1)
- U1 pad 1: Net-(R1-Pad1) -> Net-(R2-Pad1)
- U1 pad 5: Net-(R5-Pad1) -> Net-(R6-Pad1)
- U2 pad 1: VIN -> Net-(C4-Pad1)
- U2 pad 3: Net-(R4-Pad1) -> Net-(R5-Pad1)
- U2 pad 5: +3V3 -> Net-(C3-Pad1)
- U3 pad 2: Net-(C5-Pad1) -> +3V3
- U3 pad 9: IO33 -> INT
Routing:
- net INT: track 0.00 -> 35.3 mm, vias 0 -> 1
- net Net-(R1-Pad1): track 24.5 -> 0.00 mm
- net VIN: track 24.1 -> 0.00 mm, vias 2 -> 0
- net Net-(C4-Pad1): track 0.00 -> 24.1 mm, vias 0 -> 2
- net Net-(R2-Pad1): track 0.00 -> 22.8 mm
- net GND: track 106.5 -> 88.6 mm, vias 4 -> 0
- net Net-(C5-Pad1): track 15.5 -> 0.00 mm
- net Net-(C3-Pad1): track 0.00 -> 14.3 mm, vias 0 -> 2
- net IO0: track 39.5 -> 26.5 mm
- net Net-(D3-Pad1): track 8.48 -> 0.00 mm
- net Net-(D3-Pad2): track 8.26 -> 0.00 mm
- net EN: track 57.4 -> 62.2 mm
- net Net-(R4-Pad1): track 3.75 -> 0.00 mm
- net Net-(D2-Pad2): track 0.00 -> 2.36 mm
- net Net-(R6-Pad1): track 0.00 -> 2.33 mm
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Other:
- outline, holes or cut-outs redrawn
