File: clip.sch (KiCad schematic (older format))
At the start: 37 parts, among them J1 Conn_01x07, J2 BME680, J3 Moisture, J4 Conn_01x07, J5 LIS3DH, J6 Conn_01x07, J7 USB_B_Micro, J8 Conn_01x07, Q1 2.5A/30V, SW1 Switch, SW2 Switch, U1 ESP32-WROOM-32, U2 MCP73831, U3 AP2112K-3.3

Commit message: Update design
Parts:
- removed C7: 0.1uF/50V, Capacitor_SMD:C_0805_2012Metric_Pad1.15x1.40mm_HandSolder, symbol Device:C_Small
- removed J1, J6: Conn_01x07, Connector_PinHeader_2.54mm:PinHeader_1x02_P2.54mm_Vertical, symbol Connector_Generic:Conn_01x02
- added JP2: SJ, Jumper:SolderJumper-2_P1.3mm_Open_TrianglePad1.0x1.5mm, symbol Jumper:SolderJumper_2_Bridged
- D2: renamed from D5; value Yellow -> Red
- MOISTURE1: renamed from J3; value Moisture -> MOISTURE
- R6: renamed from R4; value 2.0K -> 1.0K
- USB1: renamed from J7; footprint Connector_USB:USB_Micro-B_Wuerth_614105150721_Vertical -> Connector_USB:USB_Micro-B_Wuerth_629105150521
- renumbered J2 to BME1, SW1 to BOOT1, C4 to C2, C6 to C3, C5 to C4, C2 to C5, C3 to C6, D4 to D3, D2 to D4, D3 to D5, SW2 to EN1, J8 to FLASH1, J5 to LIS1, R6 to R1, R8 to R3, R3 to R4, R7 to R5, R9 to R7, R5 to R8, R1 to R9, U2 to U1, U3 to U2, U1 to U3, J4 to VIN1
Connections:
- net IO33 is gone; now on net INT: U3.9 (IO33)
- net +3V3: now also C5.1, C6.1, U3.2 (VDD), JP2.1 (A); no longer C3.1, U2.5 (VOUT)
- net INT: now reaches LIS1.8 (Pin_8)
- net CLK: no longer names the net of U3.20 (SCK/CLK)
- net CMD: no longer names the net of U3.19 (SCS/CMD)
- net IO12: no longer names the net of U3.14 (IO12)
- net IO13: no longer names the net of U3.16 (IO13)
- net IO14: no longer names the net of U3.13 (IO14)
- net IO15: no longer names the net of U3.23 (IO15)
- net IO16: no longer names the net of U3.27 (IO16)
- net IO17: no longer names the net of U3.28 (IO17)
- net IO18: no longer names the net of U3.30 (IO18)
- net IO19: no longer names the net of U3.31 (IO19)
- net IO23: no longer names the net of U3.37 (IO23)
- net IO25: no longer names the net of U3.10 (IO25)
- net IO26: no longer names the net of U3.11 (IO26)
- net IO27: no longer names the net of U3.12 (IO27)
- net IO32: no longer names the net of U3.8 (IO32)
- net IO35: no longer names the net of U3.7 (IO35)
- net IO4: no longer names the net of U3.26 (IO4)
- net IO5: no longer names the net of U3.29 (IO5)
- net SD0: no longer names the net of U3.21 (SDO/SD0)
- net SD1: no longer names the net of U3.22 (SDI/SD1)
- net SD2: no longer names the net of U3.17 (SHD/SD2)
- net SD3: no longer names the net of U3.18 (SWP/SD3)
- net VIN: no longer names the net of C4.1, D3.1 (K), Q1.2 (S), R5.2, U2.1 (VIN)
- net VN: no longer names the net of U3.5 (SENSOR_VN)
- net VP: no longer names the net of U3.4 (SENSOR_VP)
- new net: C3.1, JP2.2 (B), U2.5 (VOUT)
- no-connect marks 10 -> 33
Other:
- note removed: "Headers\n\n"
- note removed: "Reference: NodeMCU_ESP32"
- moved on the sheet: BATTERY1, BOOT1, C1, C3, C4, C5, C6, D2, D3, D5, EN1, FLASH1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
