File: clip.sch (KiCad schematic (older format))
At the start: 35 parts, among them Q1 2.5A/30V, U1 MCP73831, U2 AP2112K-3.3, U3 ESP32-WROOM-32

Commit message: Update design
Parts:
- removed BOOT1: Switch, Button_Switch_SMD:SW_SPST_B3U-1000P-B, symbol Switch:SW_Push
- added H1, H2, H3, H4: MountingHole, MountingHole:MountingHole_2.2mm_M2_DIN965_Pad, symbol Mechanical:MountingHole
- MOISTURE1: footprint Connector_PinHeader_2.54mm:PinHeader_1x03_P2.54mm_Horizontal -> Connector_PinHeader_2.54mm:PinHeader_1x03_P2.54mm_Vertical
Connections:
- net +3V3: now also JP2.2 (B); no longer JP2.1 (A)
- net at C3.1, U2.5 (VOUT): now also JP2.1 (A); no longer JP2.2 (B)
- net IO34 renamed ADC1
Other:
- note added: "Reference: SparkFun_ESP32_Thing_Plus/Adafruit MicroLipo\nCharge current:\nI_CHG = 1000 / R_PROG\nR_PROG=1K : I_CHG=1000mA"
- note removed: "Reference: SparkFun_ESP32_Thing_Plus/Adafruit MicroLipo\nCharge current:\nI_CHG = 1000 / R_PROG\nR_PROG=2K : I_CHG=500mA"
Changed lines of the file:
@@
 $EndBitmap
 Text Notes 594  2526 0    39   ~ 0
-Reference: SparkFun_ESP32_Thing_Plus/Adafruit MicroLipo\nCharge current:\nI_CHG = 1000 / R_PROG\nR_PROG=2K : I_CHG=500mA
+Reference: SparkFun_ESP32_Thing_Plus/Adafruit MicroLipo\nCharge current:\nI_CHG = 1000 / R_PROG\nR_PROG=1K : I_CHG=1000mA
 Text Notes 3604 2510 0    39   ~ 0
 Reference: SparkFun_ESP32_Thing_Plus\nVBUS - 6V MAX\nBATT - Single Cell (4.2V MAX)
@@
 EndData
 $EndBitmap
-Text GLabel 4545 4285 0    39   Input ~ 0
-IO34
-Wire Wire Line
-	4845 4285 4545 4285
+Text GLabel 4580 4285 0    39   Input ~ 0
+ADC2
 $Comp
 L power:GND #PWR032
@@
 Wire Notes Line
 	3500 6504 6820 6504
-Wire Notes Line
-	6820 5248 6820 6504
 Text Notes 3612 5376 0    50   ~ 0
 USB-To-TTL
@@
 Connection ~ 8590 3561
 $Comp
-L Connector_Generic:Conn_01x03 MOISTURE1
+L Connector_Generic:Conn_01x04 #MOISTURE1
 U 1 1 60649048
-P 5045 4385
-F 0 "MOISTURE1" H 5125 4427 50  0000 L CNN
-F 1 "MOISTURE" H 5125 4336 50  0001 L CNN
-F 2 "Connector_PinHeader_2.54mm:PinHeader_1x03_P2.54mm_Horizontal" H 5045 4385 50  0001 C CNN
-F 3 "~" H 5045 4385 50  0001 C CNN
-	1    5045 4385
+P 5045 4285
+F 0 "#MOISTURE1" H 5125 4327 50  0000 L CNN
+F 1 "MOISTURE" H 5125 4236 50  0001 L CNN
+F 2 "Connector_PinHeader_2.54mm:PinHeader_1x04_P2.54mm_Horizontal" H 5045 4285 50  0001 C CNN
+F 3 "~" H 5045 4285 50  0001 C CNN
+	1    5045 4285
 	1    0    0    -1
 $EndComp
@@
 $EndComp
 $Comp
-L Switch:SW_Push BOOT1
+L Switch:SW_Push #BOOT1
 U 1 1 5E7E879F
 P 8340 3561
-F 0 "BOOT1" H 8340 3754 50  0000 C CNN
+F 0 "#BOOT1" H 8340 3754 50  0000 C CNN
 F 1 "Switch" H 8340 3461 50  0000 C CNN
 F 2 "Button_Switch_SMD:SW_SPST_B3U-1000P-B" H 8340 3761 50  0001 C CNN
@@
 	2650 6200 2750 6200
 Text GLabel 2750 7000 2    39   Input ~ 0
-IO34
+ADC1
 Text GLabel 2750 6300 2    39   Input ~ 0
 SCL
@@
 NoConn ~ 1450 6400
 NoConn ~ 1450 6500
-NoConn ~ 2655 7100
 NoConn ~ 2650 6800
 NoConn ~ 2650 6700
@@
 F 6 "61301811121" H 6720 1340 50  0001 C CNN "Manufacturer"
 	1    6720 1340
-	0    1    1    0
+	0    -1   -1   0
 $EndComp
 Wire Wire Line
@@
 Wire Wire Line
 	6545 4035 6295 4035
+Text GLabel 4580 4185 0    39   Input ~ 0
+ADC1
+Wire Wire Line
+	4845 4185 4580 4185
+Wire Wire Line
+	4580 4285 4845 4285
+Text GLabel 6265 4405 0    39   Input ~ 0
+ADC1
+$Comp
+L power:GND #PWR0101
+U 1 1 60C960BA
+P 6230 4705
+F 0 "#PWR0101" H 6230 4455 50  0001 C CNN
+F 1 "GND" H 6235 4532 50  0000 C CNN
+F 2 "" H 6230 4705 50  0001 C CNN
+F 3 "" H 6230 4705 50  0001 C CNN
+	1    6230 4705
+	1    0    0    -1
+$EndComp
+Wire Wire Line
+	6530 4605 6230 4605
+Wire Wire Line
+	6230 4605 6230 4705
+$Comp
+L power:+3.3V #PWR0102
+U 1 1 60C960C6
+P 5930 4505
+F 0 "#PWR0102" H 5930 4355 50  0001 C CNN
+F 1 "+3.3V" H 5945 4678 50  0000 C CNN
+F 2 "" H 5930 4505 50  0001 C CNN
+F 3 "" H 5930 4505 50  0001 C CNN
+	1    5930 4505
+	1    0    0    -1
+$EndComp
+Wire Wire Line
+	6530 4505 5930 4505
+$Comp
+L Connector_Generic:Conn_01x03 MOISTURE1
+U 1 1 60C960D1
+P 6730 4505
+F 0 "MOISTURE1" H 6810 4547 50  0000 L CNN
+F 1 "MOISTURE" H 6810 4456 50  0001 L CNN
+F 2 "Connector_PinHeader_2.54mm:PinHeader_1x03_P2.54mm_Vertical" H 6730 4505 50  0001 C CNN
+F 3 "~" H 6730 4505 50  0001 C CNN
+	1    6730 4505
+	1    0    0    -1
+$EndComp
+Wire Wire Line
+	6265 4405 6530 4405
+NoConn ~ 2650 7100
+$Comp
+L Mechanical:MountingHole H1
+U 1 1 60D3742D
+P 8165 5720
+F 0 "H1" H 8265 5766 50  0000 L CNN
+F 1 "MountingHole" H 8265 5675 50  0000 L CNN
+F 2 "MountingHole:MountingHole_2.2mm_M2_DIN965_Pad" H 8165 5720 50  0001 C CNN
+F 3 "~" H 8165 5720 50  0001 C CNN
+	1    8165 5720
+	1    0    0    -1
+$EndComp
+$Comp
+L Mechanical:MountingHole H2
+U 1 1 60D477A5
+P 7430 5720
+F 0 "H2" H 7530 5766 50  0000 L CNN
+F 1 "MountingHole" H 7530 5675 50  0000 L CNN
+F 2 "MountingHole:MountingHole_2.2mm_M2_DIN965_Pad" H 7430 5720 50  0001 C CNN
+F 3 "~" H 7430 5720 50  0001 C CNN
+	1    7430 5720
+	1    0    0    -1
+$EndComp
+$Comp
+L Mechanical:MountingHole H4
+U 1 1 60D47C68
+P 7420 6045
+F 0 "H4" H 7520 6091 50  0000 L CNN
+F 1 "MountingHole" H 7520 6000 50  0000 L CNN
+F 2 "MountingHole:MountingHole_2.2mm_M2_DIN965_Pad" H 7420 6045 50  0001 C CNN
+F 3 "~" H 7420 6045 50  0001 C CNN
+	1    7420 6045
+	1    0    0    -1
+$EndComp
+$Comp
+L Mechanical:MountingHole H3
+U 1 1 60D47E70
+P 8170 6050
+F 0 "H3" H 8270 6096 50  0000 L CNN
+F 1 "MountingHole" H 8270 6005 50  0000 L CNN
+F 2 "MountingHole:MountingHole_2.2mm_M2_DIN965_Pad" H 8170 6050 50  0001 C CNN
+F 3 "~" H 8170 6050 50  0001 C CNN
+	1    8170 6050
+	1    0    0    -1
+$EndComp
+Wire Notes Line
+	8995 5405 7140 5405
+Wire Notes Line
+	7140 5405 7140 6315
+Wire Notes Line
+	7140 6315 8995 6315
+Wire Notes Line
+	8995 5405 8995 6315
+Wire Notes Line
+	6820 5263 6820 6504
 $EndSCHEMATC

Commit message: Bump design
Connections:
- net GND: now also R4.1; no longer D4.1 (K)
- net at R2.1, U1.1 (STAT): now also D4.2 (A); no longer R4.2
- new net: D4.1 (K), R4.2
Other:
- moved on the sheet: D4, D5, R4, R8
Changed lines of the file:
@@
 L Device:LED D4
 U 1 1 5E75A88B
-P 1900 2000
-F 0 "D4" V 1950 2100 50  0000 L CNN
-F 1 "Green" V 1850 2100 50  0000 L CNN
-F 2 "LED_SMD:LED_0805_2012Metric_Pad1.15x1.40mm_HandSolder" H 1900 2000 50  0001 C CNN
-F 3 "https://katalog.we-online.de/led/datasheet/150080GS75000.pdf" H 1900 2000 50  0001 C CNN
-F 4 "732-4983-1-ND" H 1900 2000 50  0001 C CNN "Digikey"
-F 5 "https://www.digikey.de/product-detail/en/w%C3%BCrth-elektronik/150080GS75000/732-4983-1-ND/4489913" H 1900 2000 50  0001 C CNN "Digikey_link"
-F 6 "150080GS75000" H 1900 2000 50  0001 C CNN "Manufacturer"
-	1    1900 2000
+P 1900 1700
+F 0 "D4" V 1950 1800 50  0000 L CNN
+F 1 "Green" V 1850 1800 50  0000 L CNN
+F 2 "LED_SMD:LED_0805_2012Metric_Pad1.15x1.40mm_HandSolder" H 1900 1700 50  0001 C CNN
+F 3 "https://katalog.we-online.de/led/datasheet/150080GS75000.pdf" H 1900 1700 50  0001 C CNN
+F 4 "732-4983-1-ND" H 1900 1700 50  0001 C CNN "Digikey"
+F 5 "https://www.digikey.de/product-detail/en/w%C3%BCrth-elektronik/150080GS75000/732-4983-1-ND/4489913" H 1900 1700 50  0001 C CNN "Digikey_link"
+F 6 "150080GS75000" H 1900 1700 50  0001 C CNN "Manufacturer"
+	1    1900 1700
 	0    -1   -1   0
 $EndComp
@@
 L Device:R_US R4
 U 1 1 5E759248
-P 1900 1700
-F 0 "R4" H 1700 1650 50  0000 L CNN
-F 1 "1K" H 1750 1750 50  0000 L CNN
-F 2 "Resistor_SMD:R_0805_2012Metric_Pad1.15x1.40mm_HandSolder" V 1940 1690 50  0001 C CNN
-F 3 "https://industrial.panasonic.com/cdbs/www-data/pdf/RDM0000/AOA0000C307.pdf" H 1900 1700 50  0001 C CNN
-F 4 "P1.0KDACT-ND" H 1900 1700 50  0001 C CNN "Digikey"
-F 5 "https://www.digikey.de/product-detail/en/panasonic-electronic-components/ERA-6AEB102V/P1-0KDACT-ND/1465947" H 1900 1700 50  0001 C CNN "Digikey_link"
-F 6 "ERA-6AEB102V" H 1900 1700 50  0001 C CNN "Manufacturer"
-	1    1900 1700
+P 1900 2000
+F 0 "R4" H 1700 1950 50  0000 L CNN
+F 1 "1K" H 1750 2050 50  0000 L CNN
+F 2 "Resistor_SMD:R_0805_2012Metric_Pad1.15x1.40mm_HandSolder" V 1940 1990 50  0001 C CNN
+F 3 "https://industrial.panasonic.com/cdbs/www-data/pdf/RDM0000/AOA0000C307.pdf" H 1900 2000 50  0001 C CNN
+F 4 "P1.0KDACT-ND" H 1900 2000 50  0001 C CNN "Digikey"
+F 5 "https://www.digikey.de/product-detail/en/panasonic-electronic-components/ERA-6AEB102V/P1-0KDACT-ND/1465947" H 1900 2000 50  0001 C CNN "Digikey_link"
+F 6 "ERA-6AEB102V" H 1900 2000 50  0001 C CNN "Manufacturer"
+	1    1900 2000
 	-1   0    0    1
 $EndComp
@@
 Wire Wire Line
 	1650 1550 1900 1550
-Connection ~ 1900 1550
 Wire Wire Line
 	1050 1300 1050 1700
@@
 $EndComp
 Wire Wire Line
-	2757 2821 2807 2821
+	2512 3321 2562 3321
 Wire Wire Line
-	2757 2821 2757 2921
-Text GLabel 2807 2821 2    39   Input ~ 0
+	2512 3321 2512 3421
+Text GLabel 2562 3321 2    39   Input ~ 0
 IO2
 Wire Wire Line
-	2757 3221 2757 3271
+	2512 3721 2512 3771
 Wire Wire Line
-	2757 3571 2757 3621
+	2512 4071 2512 4121
 $Comp
 L power:GND #PWR027
 U 1 1 5E7F7B92
-P 2757 3621
-F 0 "#PWR027" H 2757 3371 50  0001 C CNN
-F 1 "GND" H 2762 3448 50  0000 C CNN
-F 2 "" H 2757 3621 50  0001 C CNN
-F 3 "" H 2757 3621 50  0001 C CNN
-	1    2757 3621
+P 2512 4121
+F 0 "#PWR027" H 2512 3871 50  0001 C CNN
+F 1 "GND" H 2517 3948 50  0000 C CNN
+F 2 "" H 2512 4121 50  0001 C CNN
+F 3 "" H 2512 4121 50  0001 C CNN
+	1    2512 4121
 	1    0    0    -1
 $EndComp
@@
 L Device:R_US R8
 U 1 1 5E7F7356
-P 2757 3421
-F 0 "R8" H 2825 3467 50  0000 L CNN
-F 1 "1K" H 2825 3376 50  0000 L CNN
-F 2 "Resistor_SMD:R_0805_2012Metric_Pad1.15x1.40mm_HandSolder" V 2797 3411 50  0001 C CNN
-F 3 "https://industrial.panasonic.com/cdbs/www-data/pdf/RDM0000/AOA0000C307.pdf" H 2757 3421 50  0001 C CNN
-F 4 "P1.0KDACT-ND" H 2757 3421 50  0001 C CNN "Digikey"
-F 5 "https://www.digikey.de/product-detail/en/panasonic-electronic-components/ERA-6AEB102V/P1-0KDACT-ND/1465947" H 2757 3421 50  0001 C CNN "Digikey_link"
-F 6 "ERA-6AEB102V" H 2757 3421 50  0001 C CNN "Manufacturer"
-	1    2757 3421
+P 2512 3921
+F 0 "R8" H 2580 3967 50  0000 L CNN
+F 1 "1K" H 2580 3876 50  0000 L CNN
+F 2 "Resistor_SMD:R_0805_2012Metric_Pad1.15x1.40mm_HandSolder" V 2552 3911 50  0001 C CNN
+F 3 "https://industrial.panasonic.com/cdbs/www-data/pdf/RDM0000/AOA0000C307.pdf" H 2512 3921 50  0001 C CNN
+F 4 "P1.0KDACT-ND" H 2512 3921 50  0001 C CNN "Digikey"
+F 5 "https://www.digikey.de/product-detail/en/panasonic-electronic-components/ERA-6AEB102V/P1-0KDACT-ND/1465947" H 2512 3921 50  0001 C CNN "Digikey_link"
+F 6 "ERA-6AEB102V" H 2512 3921 50  0001 C CNN "Manufacturer"
+	1    2512 3921
 	1    0    0    -1
 $EndComp
@@
 L Device:LED D5
 U 1 1 5E7F71E2
-P 2757 3071
-F 0 "D5" V 2807 3221 50  0000 L CNN
-F 1 "Blue" V 2707 3171 50  0000 L CNN
-F 2 "LED_SMD:LED_0805_2012Metric_Pad1.15x1.40mm_HandSolder" H 2757 3071 50  0001 C CNN
-F 3 "https://katalog.we-online.de/led/datasheet/150080BS75000.pdf" H 2757 3071 50  0001 C CNN
-F 4 "732-4982-1-ND" H 2757 3071 50  0001 C CNN "Digikey"
-F 5 "https://www.digikey.de/product-detail/en/w%C3%BCrth-elektronik/150080BS75000/732-4982-1-ND/4489910" H 2757 3071 50  0001 C CNN "Digikey_link"
-F 6 "150080BS75000" H 2757 3071 50  0001 C CNN "Manufacturer"
-	1    2757 3071
+P 2512 3571
+F 0 "D5" V 2562 3721 50  0000 L CNN
+F 1 "Blue" V 2462 3671 50  0000 L CNN
+F 2 "LED_SMD:LED_0805_2012Metric_Pad1.15x1.40mm_HandSolder" H 2512 3571 50  0001 C CNN
+F 3 "https://katalog.we-online.de/led/datasheet/150080BS75000.pdf" H 2512 3571 50  0001 C CNN
+F 4 "732-4982-1-ND" H 2512 3571 50  0001 C CNN "Digikey"
+F 5 "https://www.digikey.de/product-detail/en/w%C3%BCrth-elektronik/150080BS75000/732-4982-1-ND/4489910" H 2512 3571 50  0001 C CNN "Digikey_link"
+F 6 "150080BS75000" H 2512 3571 50  0001 C CNN "Manufacturer"
+	1    2512 3571
 	0    -1   -1   0
 $EndComp
@@
 Wire Notes Line
 	6820 5263 6820 6504
+Connection ~ 1900 1550
 $EndSCHEMATC
