File: test/20210701_clip.kicad_pcb (KiCad board)
At the start: 2 copper layers, 46.6 x 52.1 mm, 38 parts, among them Q1 2.5A/30V, U1 MCP73831, U2 AP2112K-3.3, U3 ESP32-WROOM-32

Commit message: Bump design
Parts:
- moved R4 34.4 mm to (158.5, 96.8), turned to 180 degrees
- moved D4 31.6 mm to (158.5, 94.5), turned to 0 degrees
- moved R2 26.8 mm to (153.8, 96.8), turned to 0 degrees
- moved D1 23.7 mm to (153.8, 94.5), turned to 180 degrees
- moved R3 15.8 mm to (163.1, 96.8), turned to 0 degrees
- moved D2 13.8 mm to (163.1, 94.5), turned to 0 degrees
- moved JP1 11.4 mm to (163.1, 91.2), turned to 180 degrees
- moved D3 9.12 mm to (145.4, 88.3)
- moved C2 8.88 mm to (147.2, 96.7)
- moved R6 8.88 mm to (147.2, 94.5)
- moved C1 8.88 mm to (139.0, 95.6)
- moved U1 8.88 mm to (142.7, 95.6)
- moved Q1 7.57 mm to (138.9, 87.6), turned to 180 degrees
- moved JP2 7.05 mm to (163.1, 88.4)
- moved C3 7.03 mm to (159.8, 87.4)
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Connections:
- D4 pad 1: Net-(D4-Pad1) -> GND
- R2 pad 1: Net-(D4-Pad2) -> Net-(R2-Pad1)
- R4 pad 1: GND -> Net-(D4-Pad2)
- R4 pad 2: Net-(D4-Pad1) -> Net-(R2-Pad1)
- U1 pad 1: Net-(D4-Pad2) -> Net-(R2-Pad1)
Routing:
- net Net-(R2-Pad1): track 0.00 -> 23.5 mm
- net Net-(D4-Pad2): track 20.0 -> 2.33 mm
- net +3V3: track 178.8 -> 168.5 mm
- net GND: track 79.5 -> 69.9 mm, vias 5 -> 7
- net VBUS: track 55.8 -> 48.1 mm, vias 4 -> 2
- net Net-(C4-Pad1): track 16.2 -> 21.8 mm
- net Net-(D4-Pad1): track 2.08 -> 0.00 mm
- net Net-(D2-Pad2): track 2.39 -> 4.34 mm
- net IO2: track 8.68 -> 7.29 mm
- net +BATT: track 23.7 -> 23.6 mm, vias 0 -> 2
